File: eagle/2WiresLink_BluePill/2WiresLink_BluePill.brd (EAGLE design)
At the start: 50.8 x 29.8 mm, 55 parts, among them IC1 TPS54060DGQ, IC3 SN74LVC1G240DBVR, IC6 TS3021ILT

Commit message: eagle: increase C21 capacity from 1nF to 10nF
In previous commit carry frequency and baud rate was decreased,
C21 capacity should be increased.
Parts:
- C21: value 1nF -> 10nF
Changed lines of the file:
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@@
 <attribute name="VALUE" x="45.638" y="15.912" size="1.27" layer="28" rot="MR270"/>
 </element>
-<element name="C21" library="rcl" library_urn="urn:adsk.eagle:library:334" package="C0603" package3d_urn="urn:adsk.eagle:package:23616/2" value="1nF" x="46.702" y="15.277" smashed="yes" rot="MR90">
+<element name="C21" library="rcl" library_urn="urn:adsk.eagle:library:334" package="C0603" package3d_urn="urn:adsk.eagle:package:23616/2" value="10nF" x="46.702" y="15.277" smashed="yes" rot="MR90">
 <attribute name="MF" value="KEMET" x="46.702" y="15.277" size="1.778" layer="28" rot="MR90" display="off"/>
-<attribute name="MPN" value="C0603C101J5GACTU" x="46.702" y="15.277" size="1.778" layer="28" rot="MR90" display="off"/>
 <attribute name="NAME" x="43.63" y="18.068" size="1.27" layer="26" rot="MR180"/>
 <attribute name="OC_FARNELL" value="unknown" x="46.702" y="15.277" size="1.778" layer="28" rot="MR90" display="off"/>
-<attribute name="OC_MOUSER" value="80-C0603C101J5G" x="46.702" y="15.277" size="1.778" layer="28" rot="MR90" display="off"/>
 <attribute name="OC_NEWARK" value="unknown" x="46.702" y="15.277" size="1.778" layer="28" rot="MR90" display="off"/>
 <attribute name="SPICEPREFIX" value="C" x="46.702" y="15.277" size="1.778" layer="28" rot="MR90" display="off"/>
